Commit message: Fixing and updating launch and config files.

File: thomas/config/robot_hardware_description.urdf (robot description, URDF)
Before this commit: robot terry, 4 links, 3 joints
Links:
- removed link base_link
- removed link front_wheel
- removed link left_wheel
- removed link right_wheel
Joints:
- removed joint PORT_A
- removed joint PORT_B
- removed joint PORT_D

Commit message: Changes to make compatible with ROS2 Jazzy.

File: thomas/config/robot_hardware_description.urdf (robot description, URDF)
Before this commit: robot charlie, 0 links, 0 joints
Links:
- added link base_link
- added link left_wheel
- added link right_wheel
Joints:
- added joint PORT_A: type continuous, parent base_link, child left_wheel
- added joint PORT_D: type continuous, parent base_link, child right_wheel
