Commit message: Adding kitt, rewritten to use its own hardware controller.

File: kitt/config/robot_hardware_description.urdf (robot description, URDF)
Before this commit: robot kitt, 4 links, 3 joints
Links:
- removed link steering_wheel
- added link steer_axis
Joints:
- removed joint PORT_A
- removed joint PORT_B
- removed joint PORT_D
- added joint left_traction_wheel: type continuous, parent base_link, child left_wheel
- added joint right_traction_wheel: type continuous, parent base_link, child right_wheel
- added joint steer_axis: type continuous, parent base_link, child steer_axis
